Commit message: update urdf for real hw

File: src/arm_description/urdf/arm.urdf.xacro (robot description, xacro)
@@ -1,21 +1,24 @@
 <?xml version="1.0"?>
 <robot xmlns:xacro="http://www.ros.org/wiki/xacro" name="cartesian_robot">
-<!-- This URDF was automatically created by SolidWorks to URDF Exporter! Originally created by Stephen Brawner (brawner@gmail.com)
+  <!-- This URDF was automatically created by SolidWorks to URDF Exporter! Originally created by
+  Stephen Brawner (brawner@gmail.com)
      Commit Version: 1.6.0-4-g7f85cfe  Build Version: 1.6.7995.38578
      For more information, please see http://wiki.ros.org/sw_urdf_exporter -->
-    <!-- Include Gazebo Parameters -->
-    <xacro:include filename="$(find arm_description)/urdf/arm_gazebo.xacro" />
-    <!-- Include ros2_control Plugins -->
-    <xacro:include filename="$(find arm_description)/urdf/arm_ros2_control.xacro" />
-    <xacro:macro name="default_transmission" params="number">
-        <transmission name="transmission${number}">
-            <plugin>transmission_interface/SimpleTransmission</plugin>
-            <actuator name="motor${number}" role="actuator1"/>
-            <joint name="joint${number}" type="prismatic" role="joint1">
-                <mechanical_reduction>1.0</mechanical_reduction>
-            </joint>
-        </transmission>
-    </xacro:macro>
-  <link name="world"/>
+  <!-- Load Simulated or Real Hardware Interfaces -->
+  <xacro:arg name="is_sim" default="true" />
+  <!-- Include Gazebo Parameters -->
+  <xacro:include filename="$(find arm_description)/urdf/arm_gazebo.xacro" />
+  <!-- Include ros2_control Plugins -->
+  <xacro:include filename="$(find arm_description)/urdf/arm_ros2_control.xacro" />
+  <xacro:macro name="default_transmission" params="number">
+    <transmission name="transmission${number}">
+      <plugin>transmission_interface/SimpleTransmission</plugin>
+      <actuator name="motor${number}" role="actuator1" />
+      <joint name="joint${number}" type="prismatic" role="joint1">
+        <mechanical_reduction>1.0</mechanical_reduction>
+      </joint>
+    </transmission>
+  </xacro:macro>
+  <link name="world" />
   <link
     name="base_link">
@@ -99,7 +102,7 @@
   </link>
   <joint name="virtual_joint" type="fixed">
-      <parent link="world"/>
-      <child link="base_link"/>
-      <origin xyz="0 0 0" rpy="0 0 0"/>
+    <parent link="world" />
+    <child link="base_link" />
+    <origin xyz="0 0 0" rpy="0 0 0" />
   </joint>
   <joint
@@ -343,7 +346,7 @@
       velocity="0.1" />
   </joint>
-    <!-- Transmissions-->
-    <xacro:default_transmission number="3"/>
-    <xacro:default_transmission number="4"/>
-    <xacro:default_transmission number="5"/>
+  <!-- Transmissions-->
+  <xacro:default_transmission number="3" />
+  <xacro:default_transmission number="4" />
+  <xacro:default_transmission number="5" />
 </robot>

File: src/arm_description/urdf/arm_ros2_control.xacro (robot description, xacro)
@@ -1,29 +1,40 @@
 <?xml version="1.0"?>
 <robot xmlns:xacro="http://www.ros.org/wiki/xacro" name="cartesian_robot">
- <ros2_control name="RobotSystem" type="system">
-  <hardware>
-    <plugin>gazebo_ros2_control/GazeboSystem</plugin>
-  </hardware>
-  <joint name="joint3">
-    <command_interface name="position">
-      <param name="min">-0.125</param>
-      <param name="max">0.120</param>
-    </command_interface>
-    <state_interface name="position"/>
-  </joint>
-  <joint name="joint4">
-    <command_interface name="position">
-      <param name="min">-0.051</param>
-      <param name="max">0.118</param>
-    </command_interface>
-    <state_interface name="position"/>
-  </joint>
-  <joint name="joint5">
-    <command_interface name="position">
-      <param name="min">-0.054</param>
-      <param name="max">0.115</param>
-    </command_interface>
-    <state_interface name="position"/>
-  </joint>
- </ros2_control>
+  <!-- Load Simulated or Real Hardware Interfaces -->
+  <xacro:arg name="is_sim" default="true" />
+  <ros2_control name="RobotSystem" type="system">
+    <xacro:if value="$(arg is_sim)">
+      <hardware>
+        <plugin>gazebo_ros2_control/GazeboSystem</plugin>
+      </hardware>
+    </xacro:if>
+    <!-- ros2_control Real Robot -->
+    <xacro:unless value="$(arg is_sim)">
+      <hardware>
+        <plugin>arm_controller/ArmInterface</plugin>
+        <param name="port">/dev/ttyACM0</param><!-- /dev/ttyUSB0 -->
+      </hardware>
+    </xacro:unless>
+    <joint name="joint3">
+      <command_interface name="position">
+        <param name="min">-0.125</param>
+        <param name="max">0.120</param>
+      </command_interface>
+      <state_interface name="position" />
+    </joint>
+    <joint name="joint4">
+      <command_interface name="position">
+        <param name="min">-0.051</param>
+        <param name="max">0.118</param>
+      </command_interface>
+      <state_interface name="position" />
+    </joint>
+    <joint name="joint5">
+      <command_interface name="position">
+        <param name="min">-0.054</param>
+        <param name="max">0.115</param>
+      </command_interface>
+      <state_interface name="position" />
+    </joint>
+  </ros2_control>
 </robot>
