Commit message: urdf change

File: src/arduinobot_description/urdf/urdfbackup/arduinobot.urdf copy.xacro (robot description, xacro)
@@ -25,5 +25,5 @@
     <inertial>
       <!-- <origin xyz="0.29184 0.032677 -0.15851" rpy="0 0 0" /> -->
-      <origin xyz="0 0 0" rpy="0 0 0" />
+      <origin xyz="0.29184 0.032677 -0.15851" rpy="0 0 0" />
       <mass
         value="0.25637" />
@@ -38,5 +38,5 @@
     <visual>
       <origin
-        xyz="-0.175 -0.183 0"
+        xyz="0 0 0"
         rpy="0 0 0" />
       <geometry>
@@ -52,5 +52,5 @@
     <collision>
       <origin
-        xyz="-0.175 -0.183 0"
+        xyz="0 0 0"
         rpy="0 0 0" />
       <geometry>
@@ -87,5 +87,5 @@
         name="">
         <color
-          rgba="1 0.94902 0.89412 1" />
+          rgba="1 0.0 0. 1" />
       </material>
     </visual>
@@ -109,5 +109,5 @@
     type="fixed">
     <!--     <origin xyz="0.1741 0.18232 0.095474" rpy="1.5708 0.0036853 0" /> -->
-    <origin xyz="0.0 0.0 0.095474" rpy="1.5708 0.0036853 0" />
+    <origin xyz="0.1741 0.18232 0.095474" rpy="1.5708 0.0036853 0" />
     <parent
       link="base_link" />
@@ -173,5 +173,4 @@
     name="x_Link">
     <inertial>
-      <!-- xyz="0.4338 -0.0037341 -0.028595" -->
       <origin
         xyz="0.4338 -0.0037341 -0.028595"
@@ -198,5 +197,5 @@
         name="">
         <color
-          rgba="1 0.0 0.0 1" />
+          rgba="1 0.94902 0.89412 1" />
       </material>
     </visual>
@@ -214,7 +213,6 @@
     name="joint3"
     type="prismatic">
-    <!-- xyz="0.4338 -0.0037341 -0.028595" -->
     <origin
-      xyz="0.5 -0.067263 0.32241"
+      xyz="0.37179 -0.067263 0.32241"
       rpy="0 1.5708 3.1416" />
     <parent
@@ -225,6 +223,6 @@
       xyz="0 0 1" />
     <limit
-      lower="0.0"
-      upper="0.240"
+      lower="-0.125"
+      upper="0.120"
       effort="1000.0"
       velocity="0.1" />
@@ -257,5 +255,5 @@
         name="">
         <color
-          rgba="0 1 0.0 1" />
+          rgba="1 0.94902 0.89412 1" />
       </material>
     </visual>
@@ -273,7 +271,6 @@
     name="joint4"
     type="prismatic">
-    <!-- xyz="0.40246 0.019644 -0.0080109" -->
     <origin
-      xyz="0.37 0.019644 -0.0080109"
+      xyz="0.40246 0.019644 -0.0080109"
       rpy="3.1416 0 0" />
     <parent
@@ -284,6 +281,6 @@
       xyz="1 0 0" />
     <limit
-      lower="0"
-      upper="0.150"
+      lower="-0.051"
+      upper="0.118"
       effort="1000.0"
       velocity="0.1" />
@@ -316,5 +313,5 @@
         name="">
         <color
-          rgba="0.0 0.0 1 1" />
+          rgba="0.79216 0.81961 0.93333 1" />
       </material>
     </visual>
@@ -333,5 +330,5 @@
     type="prismatic">
     <origin
-      xyz="0.009476 0.00 -0.070619"
+      xyz="0.009476 0.067985 -0.070619"
       rpy="0 0 -1.5708" />
     <parent
@@ -340,8 +337,8 @@
       link="z_Link" />
     <axis
-      xyz="-1 0 0" />
+      xyz="1 0 0" />
     <limit
-      lower="0"
-      upper="0.120"
+      lower="-0.054"
+      upper="0.115"
       effort="1000.0"
       velocity="0.1" />
